Commit message: Release v1.0.1: tune torso URDF parameters
Adjust mass, joint limits, and material color in dreambo_torso.urdf;
bump package version to 1.0.1.

Co-Authored-By: Claude Opus 4.7 (1M context) <noreply@anthropic.com>

File: dreambo_torso/urdf/dreambo_torso.urdf (robot description, URDF)
Before this commit: robot dreambo_torso, 8 links, 7 joints
Links:
- link base_link: mass 3.82321438743592 -> 1e-09
Joints:
- joint l_arm_pitch_joint: limit lower=0 upper=0 effort=40 velocity=10 -> lower=-3.14 upper=3.14 effort=10 velocity=1e+08
- joint l_arm_yaw_joint: limit lower=0 upper=0 effort=40 velocity=10 -> lower=-3.14 upper=3.14 effort=10 velocity=1e+08
- joint neck_pitch_joint: limit lower=0 upper=0.4 effort=27 velocity=10 -> lower=0 upper=0.4 effort=27 velocity=1e+08
- joint neck_roll_joint: limit lower=-0.4 upper=0.4 effort=27 velocity=10 -> lower=-0.4 upper=0.4 effort=27 velocity=20
- joint r_arm_pitch_joint: limit lower=0 upper=0 effort=40 velocity=10 -> lower=-3.14 upper=3.14 effort=10 velocity=1e+08
- joint r_arm_yaw_joint: limit lower=0 upper=0 effort=40 velocity=10 -> lower=-3.14 upper=3.14 effort=10 velocity=1e+08
