Commit message: Commit Dreambo Bipedal URDF

File: dreambo_bipedal/urdf/dreambo_bipedal.urdf (robot description, URDF)
Before this commit: robot dreambo_bipedal, 14 links, 13 joints
Links:
- link l_ankle_roll_link: mass 0.258324154754465 -> 0.258324154754455
- link r_ankle_pitch_link: mass 0.68752007748517 -> 0.687520077485169
- link r_ankle_roll_link: mass 0.258324154865949 -> 0.258324154865939
- link r_knee_pitch_link: mass 0.971490392039294 -> 0.971490392039295
Joints:
- joint l_ankle_roll_joint: limit lower=-0.26 upper=0.2 effort=14 velocity=37 -> lower=-0.2 upper=0.26 effort=14 velocity=37
- joint l_hip_pitch_joint: limit lower=0 upper=1.2 effort=60 velocity=20 -> lower=0 upper=1.4 effort=60 velocity=20
- joint l_knee_pitch_joint: limit lower=0 upper=1.2 effort=60 velocity=20 -> lower=-0.4 upper=2 effort=60 velocity=20
- joint r_ankle_pitch_joint: axis 0 1 0 -> 0 -1 0; origin xyz=0 0.0115 -0.09 rpy=0 0 0 -> xyz=0 -0.0115 -0.09 rpy=-3.1416 0 3.1416
- joint r_ankle_roll_joint: origin xyz=-0.0011 -0.0016 -0.070755 rpy=0 0 0 -> xyz=-0.0011 0.0016 0.070755 rpy=3.1416 0 0
- joint r_hip_pitch_joint: axis 0 -1 0 -> 0 1 0; limit lower=-1.2 upper=0 effort=60 velocity=20 -> lower=0 upper=1.4 effort=60 velocity=20; origin xyz=-0.05781 -0.02155 0 rpy=0 0 0 -> xyz=0.05781 0.02155 0 rpy=0 0 0
- joint r_hip_roll_joint: axis -1 0 0 -> 1 0 0; origin xyz=0.0579166462453084 0 -0.0679999999999469 rpy=0 0 0 -> xyz=-0.057917 0 -0.068 rpy=0 0 0
- joint r_hip_yaw_joint: origin xyz=0 -0.07 -0.006 rpy=0 0 0 -> xyz=0 -0.07 -0.006 rpy=0 0 -3.1416
- joint r_knee_pitch_joint: axis 0 1 0 -> 0 -1 0; limit lower=-1.2 upper=0 effort=60 velocity=20 -> lower=-0.4 upper=2 effort=60 velocity=20; origin xyz=0 -0.012 -0.08 rpy=0 0 0 -> xyz=0 0.012 -0.08 rpy=0 0 0

Commit message: Updates

File: dreambo_bipedal/urdf/dreambo_bipedal.urdf (robot description, URDF)
Before this commit: robot dreambo_bipedal, 14 links, 13 joints
Links:
- link r_ankle_pitch_link: mass 0.687520077485169 -> 0.68752007748517
- link r_knee_pitch_link: mass 0.971490392039295 -> 0.971490392039294
Joints:
- joint r_ankle_pitch_joint: origin xyz=0 -0.0115 -0.09 rpy=-3.1416 0 3.1416 -> xyz=0 -0.0115 -0.0900000000001102 rpy=-3.14159265358979 0 3.14159265358979
- joint r_ankle_roll_joint: origin xyz=-0.0011 0.0016 0.070755 rpy=3.1416 0 0 -> xyz=-0.00109999999999963 0.00160000000000105 0.0707548339959389 rpy=3.14159265358979 0 0
- joint r_hip_yaw_joint: origin xyz=0 -0.07 -0.006 rpy=0 0 -3.1416 -> xyz=0 -0.07 -0.006 rpy=0 0 -3.14159265358979
- joint r_knee_pitch_joint: origin xyz=0 0.012 -0.08 rpy=0 0 0 -> xyz=0 0.0119999999999999 -0.0800000000000005 rpy=0 0 0

Commit message: Update knee pitch limits

File: dreambo_bipedal/urdf/dreambo_bipedal.urdf (robot description, URDF)
Before this commit: robot dreambo_bipedal, 14 links, 13 joints
Joints:
- joint l_knee_pitch_joint: limit lower=-0.4 upper=2 effort=60 velocity=20 -> lower=-0.1 upper=2.2 effort=60 velocity=20
- joint r_knee_pitch_joint: limit lower=-0.4 upper=2 effort=60 velocity=20 -> lower=-0.1 upper=2.2 effort=60 velocity=20
