Commit message: Flip right leg joint axes for mirrored kinematics
Co-Authored-By: Claude Opus 4.7 (1M context) <noreply@anthropic.com>

File: dreambo_bipedal/urdf/dreambo_bipedal.urdf (robot description, URDF)
Before this commit: robot dreambo_bipedal, 14 links, 13 joints
Joints:
- joint r_hip_pitch_joint: axis 0 1 0 -> 0 -1 0
- joint r_hip_roll_joint: axis 1 0 0 -> -1 0 0
- joint r_knee_pitch_joint: axis 0 -1 0 -> 0 1 0

Commit message: Update hip pitch limits
Co-Authored-By: Claude Opus 4.7 (1M context) <noreply@anthropic.com>

File: dreambo_bipedal/urdf/dreambo_bipedal.urdf (robot description, URDF)
Before this commit: robot dreambo_bipedal, 14 links, 13 joints
Joints:
- joint l_hip_pitch_joint: limit lower=0 upper=1.4 effort=60 velocity=20 -> lower=-0.1 upper=1.7 effort=60 velocity=20
- joint r_hip_pitch_joint: limit lower=0 upper=1.4 effort=60 velocity=20 -> lower=-0.1 upper=1.7 effort=60 velocity=20

Commit message: Update knee and ankle pitch limits
Co-Authored-By: Claude Opus 4.7 (1M context) <noreply@anthropic.com>

File: dreambo_bipedal/urdf/dreambo_bipedal.urdf (robot description, URDF)
Before this commit: robot dreambo_bipedal, 14 links, 13 joints
Joints:
- joint l_ankle_pitch_joint: limit lower=0 upper=1.05 effort=14 velocity=37 -> lower=-0.1 upper=1.6 effort=14 velocity=37
- joint l_knee_pitch_joint: limit lower=-0.1 upper=2.2 effort=60 velocity=20 -> lower=-0.1 upper=2.6 effort=60 velocity=20
- joint r_ankle_pitch_joint: limit lower=0 upper=1.05 effort=14 velocity=37 -> lower=-0.1 upper=1.6 effort=14 velocity=37
- joint r_knee_pitch_joint: limit lower=-0.1 upper=2.2 effort=60 velocity=20 -> lower=-0.1 upper=2.6 effort=60 velocity=20
